Commit message: changed fetchbot size in the urdf to match the real fetchbot

File: src/fetchbot_description/urdf/fetchbot.urdf.xacro (robot description, xacro)
@@ -4,5 +4,5 @@
     <xacro:include filename="mobile_base.xacro" />
     <xacro:include filename="mobile_base_gazebo.xacro" />
-    <xacro:include filename="camera.xacro" />
-    <xacro:include filename="lidar.xacro" />
+    <!-- <xacro:include filename="camera.xacro" /> -->
+    <!-- <xacro:include filename="lidar.xacro" /> -->
 </robot>

File: src/fetchbot_description/urdf/mobile_base.xacro (robot description, xacro)
@@ -1,12 +1,12 @@
 <?xml version="1.0"?>
 <robot xmlns:xacro="http://www.ros.org/wiki/xacro">
-    <xacro:property name="base_length" value="0.6" />
-    <xacro:property name="base_width" value="0.4" />
-    <xacro:property name="base_height" value="0.1" />
-    <xacro:property name="wheels_base_width" value="0.05" />
-    <xacro:property name="wheel_length" value="0.05" />
-    <xacro:property name="wheel_radius" value="0.12" />
-    <xacro:property name="motor_length" value="0.02" />
-    <xacro:property name="motor_radius" value="0.05" />
+    <xacro:property name="base_length" value="0.21" />
+    <xacro:property name="base_width" value="0.19" />
+    <xacro:property name="base_height" value="0.025" />
+    <xacro:property name="wheels_base_width" value="0.015" />
+    <xacro:property name="wheel_length" value="0.02" />
+    <xacro:property name="wheel_radius" value="0.0525" />
+    <xacro:property name="motor_length" value="0.005" />
+    <xacro:property name="motor_radius" value="0.035" />
     <link name="base_footprint"/>
     <link name="base_link">
