Commit message: .

File: src/fetchbot_description/urdf/ros2_control.xacro (robot description, xacro)
@@ -21,5 +21,37 @@
             <state_interface name="position" />
         </joint>
-    </ros2_control>
+        <!-- <joint name="left_wheels_base_left_front_wheel_joint">
+            <command_interface name="velocity">
+                <param name="min">-10</param>
+                <param name="max">10</param>
+            </command_interface>
+            <state_interface name="position" />
+            <state_interface name="velocity" />
+        </joint>
+        <joint name="left_wheels_base_left_back_wheel_joint">
+            <command_interface name="velocity">
+                <param name="min">-10</param>
+                <param name="max">10</param>
+            </command_interface>
+            <state_interface name="velocity" />
+            <state_interface name="position" />
+        </joint>
+        <joint name="right_wheels_base_right_front_wheel_joint">
+            <command_interface name="velocity">
+                <param name="min">-10</param>
+                <param name="max">10</param>
+            </command_interface>
+            <state_interface name="position" />
+            <state_interface name="velocity" />
+        </joint>
+        <joint name="right_wheels_base_right_back_wheel_joint">
+            <command_interface name="velocity">
+                <param name="min">-10</param>
+                <param name="max">10</param>
+            </command_interface>
+            <state_interface name="velocity" />
+            <state_interface name="position" />
+        </joint>
+    </ros2_control> -->
     <gazebo>
         <plugin name="gazebo_ros2_control" filename="libgazebo_ros2_control.so">

Commit message: .

File: src/fetchbot_description/urdf/ros2_control.xacro (robot description, xacro)
@@ -10,6 +10,6 @@
                 <param name="max">10</param>
             </command_interface>
-            <state_interface name="position" />
-            <state_interface name="velocity" />
+            <state_interface name="velocity"/>
+            <state_interface name="position"/>
         </joint>
         <joint name="right_wheels_base_right_motor_joint">
@@ -18,6 +18,38 @@
                 <param name="max">10</param>
             </command_interface>
-            <state_interface name="velocity" />
-            <state_interface name="position" />
+            <state_interface name="velocity"/>
+            <state_interface name="position"/>
+        </joint>
+        <joint name="left_wheels_base_left_front_wheel_joint">
+            <command_interface name="velocity">
+                <param name="min">-10</param>
+                <param name="max">10</param>
+            </command_interface>
+            <state_interface name="velocity"/>
+            <state_interface name="position"/>
+        </joint>
+        <joint name="left_wheels_base_left_back_wheel_joint">
+            <command_interface name="velocity">
+                <param name="min">-10</param>
+                <param name="max">10</param>
+            </command_interface>
+            <state_interface name="velocity"/>
+            <state_interface name="position"/>
+        </joint>
+        <joint name="right_wheels_base_right_front_wheel_joint">
+            <command_interface name="velocity">
+                <param name="min">-10</param>
+                <param name="max">10</param>
+            </command_interface>
+            <state_interface name="velocity"/>
+            <state_interface name="position"/>
+        </joint>
+        <joint name="right_wheels_base_right_back_wheel_joint">
+            <command_interface name="velocity">
+                <param name="min">-10</param>
+                <param name="max">10</param>
+            </command_interface>
+            <state_interface name="velocity"/>
+            <state_interface name="position"/>
         </joint>
         <!-- <joint name="left_wheels_base_left_front_wheel_joint">
@@ -52,6 +84,6 @@
             <state_interface name="velocity" />
             <state_interface name="position" />
-        </joint>
-    </ros2_control> -->
+        </joint>-->
+    </ros2_control>
     <gazebo>
         <plugin name="gazebo_ros2_control" filename="libgazebo_ros2_control.so">

Commit message: .

File: src/fetchbot_description/urdf/ros2_control.xacro (robot description, xacro)
@@ -5,4 +5,5 @@
             <plugin>gazebo_ros2_control/GazeboSystem</plugin>
         </hardware>
+        <!-- left motor -->
         <joint name="left_wheels_base_left_motor_joint">
             <command_interface name="velocity">
@@ -13,4 +14,5 @@
             <state_interface name="position"/>
         </joint>
+        <!-- right motor -->
         <joint name="right_wheels_base_right_motor_joint">
             <command_interface name="velocity">
@@ -21,4 +23,5 @@
             <state_interface name="position"/>
         </joint>
+        <!-- left front wheel -->
         <joint name="left_wheels_base_left_front_wheel_joint">
             <command_interface name="velocity">
@@ -29,4 +32,5 @@
             <state_interface name="position"/>
         </joint>
+        <!-- left back wheel -->
         <joint name="left_wheels_base_left_back_wheel_joint">
             <command_interface name="velocity">
@@ -37,4 +41,5 @@
             <state_interface name="position"/>
         </joint>
+        <!-- right front wheel -->
         <joint name="right_wheels_base_right_front_wheel_joint">
             <command_interface name="velocity">
@@ -45,4 +50,5 @@
             <state_interface name="position"/>
         </joint>
+        <!-- right back wheel -->
         <joint name="right_wheels_base_right_back_wheel_joint">
             <command_interface name="velocity">
@@ -53,43 +59,14 @@
             <state_interface name="position"/>
         </joint>
-        <!-- <joint name="left_wheels_base_left_front_wheel_joint">
-            <command_interface name="velocity">
-                <param name="min">-10</param>
-                <param name="max">10</param>
-            </command_interface>
-            <state_interface name="position" />
-            <state_interface name="velocity" />
-        </joint>
-        <joint name="left_wheels_base_left_back_wheel_joint">
-            <command_interface name="velocity">
-                <param name="min">-10</param>
-                <param name="max">10</param>
-            </command_interface>
-            <state_interface name="velocity" />
-            <state_interface name="position" />
-        </joint>
-        <joint name="right_wheels_base_right_front_wheel_joint">
-            <command_interface name="velocity">
-                <param name="min">-10</param>
-                <param name="max">10</param>
-            </command_interface>
-            <state_interface name="position" />
-            <state_interface name="velocity" />
-        </joint>
-        <joint name="right_wheels_base_right_back_wheel_joint">
-            <command_interface name="velocity">
-                <param name="min">-10</param>
-                <param name="max">10</param>
-            </command_interface>
-            <state_interface name="velocity" />
-            <state_interface name="position" />
-        </joint>-->
     </ros2_control>
     <gazebo>
-        <plugin name="gazebo_ros2_control" filename="libgazebo_ros2_control.so">
+        <plugin filename="libgazebo_ros2_control.so" name="gazebo_ros2_control">
+            <robot_param>robot_description</robot_param>
+            <robot_param_node>robot_state_publisher</robot_param_node>
             <parameters>$(find fetchbot_description)/config/my_controllers.yaml</parameters>
+            <controller_manager_name>simulation_controller_manager</controller_manager_name>
         </plugin>
     </gazebo>
-        <gazebo reference="base_link">
+    <gazebo reference="base_link">
         <material>Gazebo/Grey</material>
     </gazebo>
