Commit message: work in progress

File: src/fetchbot_description/urdf/mobile_base.xacro (robot description, xacro)
@@ -81,5 +81,5 @@
             <collision>
                 <geometry>
-                    <cylinder radius="${wheel_radius}" length="${wheel_length}"/>
+                    <sphere radius="${wheel_radius}" />
                 </geometry>
                 <origin xyz="0 0 0" rpy="${pi / 2.0} 0 0"/>

File: src/fetchbot_description/urdf/ros2_control.xacro (robot description, xacro)
@@ -86,13 +86,21 @@
     <gazebo reference="left_front_wheel_link">
         <material>Gazebo/Blue</material>
+        <mu1 value="1"/>
+        <mu2 value="1"/>
     </gazebo>
     <gazebo reference="left_back_wheel_link">
         <material>Gazebo/Blue</material>
+        <mu1 value="1"/>
+        <mu2 value="1"/>
     </gazebo>
     <gazebo reference="right_front_wheel_link">
         <material>Gazebo/Blue</material>
+        <mu1 value="1"/>
+        <mu2 value="1"/>
     </gazebo>
     <gazebo reference="right_back_wheel_link">
         <material>Gazebo/Blue</material>
+        <mu1 value="1"/>
+        <mu2 value="1"/>
     </gazebo>
 </robot>
