Commit message: updated ros2 control

File: src/fetchbot_description/urdf/gazebo_controller.xacro (robot description, xacro)
@@ -2,29 +2,17 @@
 <robot xmlns:xacro="http://www.ros.org/wiki/xacro">
     <gazebo reference="base_link">
-        <material>Gazebo/Grey</material>
+        <material>Gazebo/Blue</material>
     </gazebo>
-    <gazebo reference="left_wheels_base_link">
+    <gazebo reference="left_front_wheel_link">
         <material>Gazebo/Red</material>
     </gazebo>
-    <gazebo reference="right_wheels_base_link">
+    <gazebo reference="left_back_wheel_link">
+        <material>Gazebo/Red</material>
+    </gazebo>
+    <gazebo reference="right_front_wheel_link">
         <material>Gazebo/Green</material>
     </gazebo>
-    <gazebo reference="left_motor_link">
-        <material>Gazebo/Purple</material>
-    </gazebo>
-    <gazebo reference="right_motor_link">
-        <material>Gazebo/Purple</material>
-    </gazebo>
-    <gazebo reference="left_front_wheel_link">
-        <material>Gazebo/Blue</material>
-    </gazebo>
-    <gazebo reference="left_back_wheel_link">
-        <material>Gazebo/Blue</material>
-    </gazebo>
-    <gazebo reference="right_front_wheel_link">
-        <material>Gazebo/Blue</material>
-    </gazebo>
     <gazebo reference="right_back_wheel_link">
-        <material>Gazebo/Blue</material>
+        <material>Gazebo/Green</material>
     </gazebo>
     <gazebo>
@@ -34,10 +22,8 @@
             <!-- wheels -->
             <num_wheel_pairs>3</num_wheel_pairs>
-            <left_joint>left_wheels_base_left_motor_joint</left_joint>
-            <left_joint>left_wheels_base_left_front_wheel_joint</left_joint>
-            <left_joint>left_wheels_base_left_back_wheel_joint</left_joint>
-            <right_joint>right_wheels_base_right_motor_joint</right_joint>
-            <right_joint>right_wheels_base_right_front_wheel_joint</right_joint>
-            <right_joint>right_wheels_base_right_back_wheel_joint</right_joint>
+            <left_joint>left_front_wheel_joint</left_joint>
+            <left_joint>left_back_wheel_joint</left_joint>
+            <right_joint>right_front_wheel_joint</right_joint>
+            <right_joint>right_back_wheel_joint</right_joint>
             <!-- kinematics -->
             <wheel_separation>${base_width + wheel_length}</wheel_separation>

File: src/fetchbot_description/urdf/mobile_base.xacro (robot description, xacro)
@@ -2,11 +2,11 @@
 <robot xmlns:xacro="http://www.ros.org/wiki/xacro">
     <xacro:property name="base_length" value="0.21" />
-    <xacro:property name="base_width" value="0.19" />
+    <xacro:property name="base_width" value="0.21" />
     <xacro:property name="base_height" value="0.025" />
-    <xacro:property name="wheels_base_width" value="0.015" />
-    <xacro:property name="wheel_length" value="0.02" />
+    <xacro:property name="wheel_length" value="0.025" />
     <xacro:property name="wheel_radius" value="0.0525" />
-    <xacro:property name="motor_length" value="0.005" />
-    <xacro:property name="motor_radius" value="0.035" />
+    <xacro:property name="wheel_separation" value="0.125" />
+    <xacro:property name="wheel_mass" value="2.0" />
+    <xacro:property name="base_mass" value="10.0" />
     <link name="base_footprint"/>
     <link name="base_link">
@@ -17,5 +17,5 @@
             </geometry>
             <origin xyz="0 0 ${base_height / 2.0}" rpy="0 0 0"/>
-            <material name="grey"/>
+            <material name="blue"/>
         </visual>
         <collision>
@@ -25,50 +25,8 @@
             <origin xyz="0 0 ${base_height / 2.0}" rpy="0 0 0"/>
         </collision>
-        <xacro:box_inertia m="2.0" l="${base_length}" w="${base_width}" h="${base_height}"
+        <xacro:box_inertia m="${base_mass}" l="${base_length}" w="${base_width}" h="${base_height}"
                            xyz="0 0 ${base_height / 2.0}" rpy="0 0 0" />
     </link>
-    <xacro:macro name="wheels_base_link" params="prefix direction color">
-        <link name="${prefix}_wheels_base_link">
-            <visual>
-                <geometry>
-                    <box size="${base_length} ${wheels_base_width} ${base_height}"/>
-                </geometry>
-                <origin xyz="0 ${direction * wheels_base_width / 2.0} 0" rpy="0 0 0"/>
-                <material name="${color}"/>
-            </visual>
-            <collision>
-                <geometry>
-                    <box size="${base_length} ${wheels_base_width} ${base_height}"/>
-                </geometry>
-                <origin xyz="0 ${direction * wheels_base_width / 2.0} 0" rpy="0 0 0"/>
-            </collision>
-            <xacro:box_inertia m="0.3" l="${base_length}" w="${wheels_base_width}" h="${base_height}"
-                            xyz="0 ${direction * wheels_base_width / 2.0} 0" rpy="0 0 0"/>
-        </link>
-    </xacro:macro>
-    <xacro:wheels_base_link prefix="left" direction="1" color="red" />
-    <xacro:wheels_base_link prefix="right" direction="-1" color="green" />
-    <xacro:macro name="motor_link" params="prefix">
-        <link name="${prefix}_motor_link">
-            <visual>
-                <geometry>
-                    <cylinder radius="${motor_radius}" length="${motor_length}"/>
-                </geometry>
-                <origin xyz="0 0 0" rpy="${pi / 2.0} 0 0"/>
-                <material name="purple"/>
-            </visual>
-            <collision>
-                <geometry>
-                    <cylinder radius="${motor_radius}" length="${motor_length}"/>
-                </geometry>
-                <origin xyz="0 0 0" rpy="${pi / 2.0} 0 0"/>
-            </collision>
-             <xacro:cylinder_inertia m="0.1" r="${motor_radius}" h="${motor_length}"
-                            xyz="0 0 0" rpy="${pi / 2.0} 0 0"/>
-        </link>
-    </xacro:macro>
-    <xacro:motor_link prefix="left" />
-    <xacro:motor_link prefix="right" />
-    <xacro:macro name="wheel_link" params="prefix">
+    <xacro:macro name="wheel_link" params="prefix color">
         <link name="${prefix}_wheel_link">
             <visual>
@@ -77,20 +35,21 @@
                 </geometry>
                 <origin xyz="0 0 0" rpy="${pi / 2.0} 0 0"/>
-                <material name="blue"/>
+                <material name="${color}"/>
             </visual>
             <collision>
                 <geometry>
-                    <sphere radius="${wheel_radius}" />
+                    <!-- <cylinder radius="${wheel_radius}" length="${wheel_length}"/> -->
+                    <sphere radius="${wheel_radius}"/>
                 </geometry>
                 <origin xyz="0 0 0" rpy="${pi / 2.0} 0 0"/>
             </collision>
-             <xacro:cylinder_inertia m="0.1" r="${wheel_radius}" h="${wheel_length}"
+            <xacro:cylinder_inertia m="${wheel_mass}" r="${wheel_radius}" h="${wheel_length}"
                             xyz="0 0 0" rpy="${pi / 2.0} 0 0"/>
         </link>
     </xacro:macro>
-    <xacro:wheel_link prefix="left_front" />
-    <xacro:wheel_link prefix="left_back" />
-    <xacro:wheel_link prefix="right_front" />
-    <xacro:wheel_link prefix="right_back" />
+    <xacro:wheel_link prefix="left_front" color="green" />
+    <xacro:wheel_link prefix="left_back" color="green" />
+    <xacro:wheel_link prefix="right_front" color="red" />
+    <xacro:wheel_link prefix="right_back" color="red"/>
     <joint name="base_joint" type="fixed">
         <parent link="base_footprint"/>
@@ -98,35 +57,24 @@
         <origin xyz="0 0 ${wheel_radius - (base_height / 2.0)}" rpy="0 0 0"/>
     </joint>
-    <xacro:macro name="base_wheels_base_joint" params="prefix direction">
-        <joint name="base_${prefix}_wheels_base_joint" type="fixed">
+    <xacro:macro name="front_wheel_joint" params="prefix1 direction1 direction2">
+        <joint name="${prefix1}_front_wheel_joint" type="continuous">
             <parent link="base_link"/>
-            <child link="${prefix}_wheels_base_link"/>
-            <origin xyz="0 ${direction * base_width / 2.0} ${base_height / 2.0}" rpy="0 0 0"/>
-        </joint>
-    </xacro:macro>
-    <xacro:base_wheels_base_joint prefix="left" direction="1" />
-    <xacro:base_wheels_base_joint prefix="right" direction="-1" />
-    <xacro:macro name="wheels_base_motor_joint" params="prefix direction">
-        <joint name="${prefix}_wheels_base_${prefix}_motor_joint" type="continuous">
-            <parent link="${prefix}_wheels_base_link"/>
-            <child link="${prefix}_motor_link"/>
-            <origin xyz="0 ${direction * (wheels_base_width + (motor_length / 2.0))} 0" rpy="0 0 0"/>
+            <child link="${prefix1}_front_wheel_link"/>
+            <origin xyz="${direction1 * (wheel_separation / 2.0)} ${direction2 * ((base_width + wheel_length) / 2.0)} 0" rpy="0 0 0"/>
             <axis xyz="0 1 0"/>
         </joint>
     </xacro:macro>
-    <xacro:wheels_base_motor_joint prefix="left" direction="1" />
-    <xacro:wheels_base_motor_joint prefix="right" direction="-1" />
-    <xacro:macro name="wheels_base_wheel_joint" params="prefix1 prefix2 direction1 direction2">
-        <joint name="${prefix1}_wheels_base_${prefix1}_${prefix2}_wheel_joint" type="continuous">
-            <parent link="${prefix1}_wheels_base_link"/>
-            <child link="${prefix1}_${prefix2}_wheel_link"/>
-            <origin xyz="${direction1 * (motor_radius + wheel_radius)} ${direction2 * (wheels_base_width + (wheel_length / 2.0))} 0" rpy="0 0 0"/>
+    <xacro:front_wheel_joint prefix1="left" direction1="1" direction2="1" />
+    <xacro:front_wheel_joint prefix1="right" direction1="1" direction2="-1" />
+    <xacro:macro name="back_wheel_joint" params="prefix1 direction1 direction2">
+        <joint name="${prefix1}_back_wheel_joint" type="continuous">
+            <parent link="base_link"/>
+            <child link="${prefix1}_back_wheel_link"/>
+            <origin xyz="${direction1 * (wheel_separation / 2.0)} ${direction2 * ((base_width + wheel_length) / 2.0)} 0" rpy="0 0 0"/>
             <axis xyz="0 1 0"/>
-            <mimic joint="${prefix1}_wheels_base_${prefix1}_motor_joint" multiplier="1" offset="0"/>
+            <mimic joint="${prefix1}_front_wheel_joint" multiplier="1" offset="0"/>
         </joint>
     </xacro:macro>
-    <xacro:wheels_base_wheel_joint prefix1="left" prefix2="front" direction1="1" direction2="1" />
-    <xacro:wheels_base_wheel_joint prefix1="left" prefix2="back" direction1="-1" direction2="1" />
-    <xacro:wheels_base_wheel_joint prefix1="right" prefix2="front" direction1="1" direction2="-1" />
-    <xacro:wheels_base_wheel_joint prefix1="right" prefix2="back" direction1="-1" direction2="-1" />
+    <xacro:back_wheel_joint prefix1="left" direction1="-1" direction2="1" />
+    <xacro:back_wheel_joint prefix1="right" direction1="-1" direction2="-1" />
 </robot>

File: src/fetchbot_description/urdf/ros2_control.xacro (robot description, xacro)
@@ -5,24 +5,6 @@
             <plugin>gazebo_ros2_control/GazeboSystem</plugin>
         </hardware>
-        <!-- left motor -->
-        <joint name="left_wheels_base_left_motor_joint">
-            <command_interface name="velocity">
-                <param name="min">-10</param>
-                <param name="max">10</param>
-            </command_interface>
-            <state_interface name="velocity"/>
-            <state_interface name="position"/>
-        </joint>
-        <!-- right motor -->
-        <joint name="right_wheels_base_right_motor_joint">
-            <command_interface name="velocity">
-                <param name="min">-10</param>
-                <param name="max">10</param>
-            </command_interface>
-            <state_interface name="velocity"/>
-            <state_interface name="position"/>
-        </joint>
         <!-- left front wheel -->
-        <joint name="left_wheels_base_left_front_wheel_joint">
+        <joint name="left_front_wheel_joint">
             <command_interface name="velocity">
                 <param name="min">-10</param>
@@ -33,5 +15,5 @@
         </joint>
         <!-- left back wheel -->
-        <joint name="left_wheels_base_left_back_wheel_joint">
+        <joint name="left_back_wheel_joint">
             <command_interface name="velocity">
                 <param name="min">-10</param>
@@ -42,5 +24,5 @@
         </joint>
         <!-- right front wheel -->
-        <joint name="right_wheels_base_right_front_wheel_joint">
+        <joint name="right_front_wheel_joint">
             <command_interface name="velocity">
                 <param name="min">-10</param>
@@ -51,5 +33,5 @@
         </joint>
         <!-- right back wheel -->
-        <joint name="right_wheels_base_right_back_wheel_joint">
+        <joint name="right_back_wheel_joint">
             <command_interface name="velocity">
                 <param name="min">-10</param>
@@ -70,37 +52,17 @@
     </gazebo>
     <gazebo reference="base_link">
-        <material>Gazebo/Grey</material>
+        <material>Gazebo/Blue</material>
     </gazebo>
-    <gazebo reference="left_wheels_base_link">
+    <gazebo reference="left_front_wheel_link">
+        <material>Gazebo/Green</material>
+    </gazebo>
+    <gazebo reference="left_back_wheel_link">
+        <material>Gazebo/Green</material>
+    </gazebo>
+    <gazebo reference="right_front_wheel_link">
         <material>Gazebo/Red</material>
     </gazebo>
-    <gazebo reference="right_wheels_base_link">
-        <material>Gazebo/Green</material>
-    </gazebo>
-    <gazebo reference="left_motor_link">
-        <material>Gazebo/Purple</material>
-    </gazebo>
-    <gazebo reference="right_motor_link">
-        <material>Gazebo/Purple</material>
-    </gazebo>
-    <gazebo reference="left_front_wheel_link">
-        <material>Gazebo/Blue</material>
-        <mu1 value="1"/>
-        <mu2 value="1"/>
-    </gazebo>
-    <gazebo reference="left_back_wheel_link">
-        <material>Gazebo/Blue</material>
-        <mu1 value="1"/>
-        <mu2 value="1"/>
-    </gazebo>
-    <gazebo reference="right_front_wheel_link">
-        <material>Gazebo/Blue</material>
-        <mu1 value="1"/>
-        <mu2 value="1"/>
-    </gazebo>
     <gazebo reference="right_back_wheel_link">
-        <material>Gazebo/Blue</material>
-        <mu1 value="1"/>
-        <mu2 value="1"/>
+        <material>Gazebo/Red</material>
     </gazebo>
 </robot>
