Commit message: update lidar size in the urdf to match real robot

File: src/fetchbot_description/urdf/lidar.xacro (robot description, xacro)
@@ -2,5 +2,5 @@
 <robot xmlns:xacro="http://www.ros.org/wiki/xacro">
     <xacro:property name="lidar_radius" value="0.05" />
-    <xacro:property name="lidar_length" value="0.1" />
+    <xacro:property name="lidar_length" value="0.0725" />
     <joint name="laser_joint" type="fixed">
         <parent link="base_link"/>
