Commit message: update urdf files

File: fetchbot_description/urdf/fetchbot.urdf.xacro (robot description, xacro)
@@ -3,5 +3,4 @@
     <xacro:include filename="common_properties.xacro" />
     <xacro:include filename="mobile_base.xacro" />
-    <!-- <xacro:include filename="mobile_base_gazebo.xacro" /> -->
     <xacro:include filename="ros2_control_gazebo.xacro" />
     <!-- <xacro:include filename="diffdrive.ros2_control.xacro" /> -->

File: fetchbot_description/urdf/mobile_base.xacro (robot description, xacro)
@@ -39,6 +39,6 @@
             <collision>
                 <geometry>
-                    <!-- <cylinder radius="${wheel_radius}" length="${wheel_length}"/> -->
-                    <sphere radius="${wheel_radius}"/>
+                    <cylinder radius="${wheel_radius}" length="${wheel_length}"/>
+                    <!-- <sphere radius="${wheel_radius}"/> -->
                 </geometry>
                 <origin xyz="0 0 0" rpy="${pi / 2.0} 0 0"/>
