Commit message: update lidar pos in the urdf

File: fetchbot_description/urdf/lidar.xacro (robot description, xacro)
@@ -1,10 +1,10 @@
 <?xml version="1.0"?>
 <robot xmlns:xacro="http://www.ros.org/wiki/xacro">
-    <xacro:property name="lidar_radius" value="0.05" />
+    <xacro:property name="lidar_radius" value="0.025" />
     <xacro:property name="lidar_length" value="0.0725" />
     <joint name="laser_joint" type="fixed">
         <parent link="base_link"/>
         <child link="laser_link"/>
-        <origin xyz="0 0 ${base_height + lidar_length}" rpy="0 0 0"/>
+        <origin xyz="0.025 0 ${base_height + lidar_length}" rpy="0 0 0"/>
     </joint>
     <link name="laser_link">
