Commit message: added a fake claw to the robot urdf and updated camera and lidar size and pos

File: fetchbot_description/urdf/camera.xacro (robot description, xacro)
@@ -2,6 +2,7 @@
 <robot xmlns:xacro="http://www.ros.org/wiki/xacro">
     <xacro:property name="camera_length" value="0.01" />
-    <xacro:property name="camera_width" value="0.1" />
-    <xacro:property name="camera_height" value="0.05" />
+    <xacro:property name="camera_width" value="0.04" />
+    <xacro:property name="camera_height" value="0.04" />
+    <xacro:property name="M_PI" value="3.1415926535897931" />
     <link name="camera_link">
         <visual>
@@ -20,7 +21,8 @@
     </link>
     <joint name="base_camera_joint" type="fixed">
-        <parent link="base_link" />
+        <parent link="claw_link" />
         <child link="camera_link" />
-        <origin xyz="${(camera_length + base_length) / 2.0} 0 ${base_height / 2.0}" rpy="0 0 0" />
+        <origin xyz="${claw_length / 4.0} 0 ${(claw_height+
+         camera_height) / 2.0}" rpy="0 0 0" />
     </joint>
     <link name="camera_link_optical">
@@ -37,8 +39,22 @@
         <material>Gazebo/White</material>
         <sensor name="camera_sensor" type="camera">
-            <pose>0 0 0 0 0 0</pose>
-            <visualize>true</visualize>
-            <update_rate>10.0</update_rate>
+            <update_rate>30.0</update_rate>
+            <camera>
+                <!-- <pose>0.035 0 0.078 0 ${-M_PI/2} 0</pose> -->
+                <!-- <pose>0.0 0 0.0 0 0.0 0</pose> -->
+                <horizontal_fov>${45 * M_PI/180.0}</horizontal_fov>
+                <image>
+                    <!-- <format>R8G8B8</format> -->
+                    <width>640</width>
+                    <height>480</height>
+                </image>
+                <!-- <clip>
+                    <near>0.01</near>
+                    <far>100</far>
+                </clip> -->
+            </camera>
             <plugin name="camera_controller" filename="libgazebo_ros_camera.so">
+                <alwaysOn>true</alwaysOn>
+                <updateRate>0.0</updateRate>
                 <frame_name>camera_link_optical</frame_name>
             </plugin>

File: fetchbot_description/urdf/fetchbot.urdf.xacro (robot description, xacro)
@@ -6,4 +6,5 @@
     <!-- <xacro:include filename="diffdrive.ros2_control.xacro" /> -->
     <xacro:include filename="lidar.xacro" />
+    <xacro:include filename="claw.xacro" />
     <xacro:include filename="camera.xacro" />
 </robot>

File: fetchbot_description/urdf/lidar.xacro (robot description, xacro)
@@ -1,6 +1,6 @@
 <?xml version="1.0"?>
 <robot xmlns:xacro="http://www.ros.org/wiki/xacro">
-    <xacro:property name="lidar_radius" value="0.025" />
-    <xacro:property name="lidar_length" value="0.0725" />
+    <xacro:property name="lidar_radius" value="0.035" />
+    <xacro:property name="lidar_length" value="0.117" />
     <joint name="laser_joint" type="fixed">
         <parent link="base_link"/>

File: fetchbot_description/urdf/mobile_base.xacro (robot description, xacro)
@@ -3,5 +3,5 @@
     <xacro:property name="base_length" value="0.21" />
     <xacro:property name="base_width" value="0.21" />
-    <xacro:property name="base_height" value="0.025" />
+    <xacro:property name="base_height" value="0.026" />
     <xacro:property name="wheel_length" value="0.025" />
     <xacro:property name="wheel_radius" value="0.0525" />

Commit message: update camera pos and angle on the urdf

File: fetchbot_description/urdf/camera.xacro (robot description, xacro)
@@ -42,5 +42,5 @@
             <camera>
                 <!-- <pose>0.035 0 0.078 0 ${-M_PI/2} 0</pose> -->
-                <!-- <pose>0.0 0 0.0 0 0.0 0</pose> -->
+                <pose>0 0 0 0 -0.05 0</pose>
                 <horizontal_fov>${45 * M_PI/180.0}</horizontal_fov>
                 <image>
@@ -49,8 +49,8 @@
                     <height>480</height>
                 </image>
-                <!-- <clip>
+                <clip>
                     <near>0.01</near>
                     <far>100</far>
-                </clip> -->
+                </clip>
             </camera>
             <plugin name="camera_controller" filename="libgazebo_ros_camera.so">

File: fetchbot_description/urdf/claw.xacro (robot description, xacro)
@@ -65,5 +65,5 @@
         <parent link="base_link" />
         <child link="claw_link" />
-        <origin xyz="${(claw_length + base_length) / 2.0} 0 ${claw_height / 2.0}" rpy="0 0 0" />
+        <origin xyz="${(claw_length + base_length) / 2.0} 0 ${-claw_height / 2.0}" rpy="0 0 0" />
     </joint>
 </robot>
