Commit message: added color to the claw and removed sensor visualize in gazebo

File: fetchbot_description/urdf/claw.xacro (robot description, xacro)
@@ -12,5 +12,5 @@
                 <box size="${claw_length} ${claw_width} ${claw_height}" />
             </geometry>
-            <material name="white" />
+            <material name="purple" />
         </visual>
         <collision>
@@ -27,5 +27,5 @@
                 <box size="${gripper_length} ${gripper_width} ${gripper_height}" />
             </geometry>
-            <material name="white" />
+            <material name="purple" />
         </visual>
         <collision>
@@ -42,5 +42,5 @@
                 <box size="${gripper_length} ${gripper_width} ${gripper_height}" />
             </geometry>
-            <material name="white" />
+            <material name="purple" />
         </visual>
         <collision>

File: fetchbot_description/urdf/lidar.xacro (robot description, xacro)
@@ -28,5 +28,5 @@
         <sensor name="laser" type="ray">
             <pose> 0 0 0 0 0 0 </pose>
-            <visualize>true</visualize>
+            <visualize>false</visualize>
             <update_rate>10</update_rate>
             <ray>

File: fetchbot_description/urdf/ros2_control_gazebo.xacro (robot description, xacro)
@@ -66,3 +66,12 @@
         <material>Gazebo/Red</material>
     </gazebo>
+    <gazebo reference="claw_link">
+        <material>Gazebo/Purple</material>
+    </gazebo>
+    <gazebo reference="left_gripper_link">
+        <material>Gazebo/Purple</material>
+    </gazebo>
+    <gazebo reference="right_gripper_link">
+        <material>Gazebo/Purple</material>
+    </gazebo>
 </robot>

Commit message: added launch files

File: fetchbot_description/urdf/claw.xacro (robot description, xacro)
@@ -4,5 +4,5 @@
     <xacro:property name="claw_width" value="0.15" />
     <xacro:property name="claw_height" value="0.013" />
-    <xacro:property name="gripper_length" value="0.07" />
+    <xacro:property name="gripper_length" value="0.045" />
     <xacro:property name="gripper_width" value="0.03" />
     <xacro:property name="gripper_height" value="0.013" />
